File: Kicad/X1_EMM.kicad_pcb (KiCad board)
At the start: 2 copper layers, 137 x 140.7 mm, 46 parts, among them J1 for Card-Slot, U1 74LS04, U10 74LS193, U11 74LS193, U12 74LS138, U13 74LS138, U14 HM628512LFP-5, U15 74LS11, U16 74LS245, U2 74LS04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

Commit message: Add files via upload
Parts:
- added C19: 0.1uF, Capacitor_THT:C_Rect_L4.0mm_W2.5mm_P2.50mm, F.Cu at (63.7, 154.6)
- added D3: 1S4, Diode_THT:D_DO-41_SOD81_P10.16mm_Horizontal, F.Cu at (104.9, 162.2)
- added R3: 10k, Resistor_THT:R_Axial_DIN0207_L6.3mm_D2.5mm_P7.62mm_Horizontal, F.Cu at (119.5, 152.7)
- added S3: SLIDE_SWITCH_3P, Connector_PinHeader_2.54mm:PinHeader_1x03_P2.54mm_Vertical, F.Cu at (96.7, 193.9)
- added U17: 74LS04, Package_DIP:DIP-14_W7.62mm_LongPads, F.Cu at (66.8, 159.7)
- moved D2 11.7 mm to (104.9, 169.8)
- moved D1 11.7 mm to (104.9, 176.8)
- moved BT1 8.91 mm to (81.4, 176.8)
- moved C12 1.27 mm to (136.7, 138.1)
- moved C17 1.27 mm to (155.1, 106.9)
- moved C2 1.27 mm to (139.2, 94.2)
- moved C5 1.27 mm to (139.2, 117.1)
- moved C13 1.27 mm to (33.2, 154.6)
- moved C16 1.27 mm to (33.2, 117.1)
- moved C6 1.27 mm to (33.2, 94.2)
- moved C8 1.27 mm to (33.2, 138.1)
- moved U13 1.27 mm to (36.4, 159.7)
- moved U16 1.27 mm to (36.4, 122.2)
- moved U6 1.27 mm to (36.4, 99.3)
- moved U8 1.27 mm to (36.4, 143.1)
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Connections:
- U12 pad 4: Net-(R2-Pad2) -> Net-(U12-Pad4)
- U12 pad 5: Net-(R2-Pad2) -> Net-(U12-Pad4)
- U13 pad 4: Net-(R2-Pad2) -> Net-(U12-Pad4)
- U13 pad 5: Net-(R2-Pad2) -> Net-(U12-Pad4)
- U14 pad 29: /x3_WR -> Net-(R3-Pad2)
- U4 pad 8: Net-(R2-Pad2) -> Net-(U12-Pad4)
Routing:
- net Net-(U12-Pad4): track 0.00 -> 161.3 mm, vias 0 -> 1
- net Net-(R2-Pad2): track 194.5 -> 100.8 mm, vias 0 -> 3
- net Net-(R3-Pad2): track 0.00 -> 60.4 mm
- net /x3_WR: track 116.8 -> 79.6 mm
- net Net-(D3-Pad1): track 0.00 -> 35.2 mm
- net GND: track 723.3 -> 755.7 mm
- net Net-(U10-Pad1): track 124.0 -> 97.0 mm, vias 2 -> 3
- net Net-(D3-Pad2): track 0.00 -> 22.8 mm
- net Net-(U14-Pad15): track 163.8 -> 142.2 mm, vias 0 -> 1
- net +5V: track 533.6 -> 554.9 mm, vias 1 -> 0
- net Net-(U14-Pad18): track 126.0 -> 146.7 mm, vias 1 -> 0
- net /A0: track 228.5 -> 210.0 mm, vias 0 -> 1
- net /~WR: track 122.2 -> 138.3 mm, vias 1 -> 0
- net Net-(U14-Pad21): track 110.7 -> 122.2 mm
- net /A1: track 226.5 -> 215.4 mm
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Other:
- board text added: "EMM for X1 Rev1.5"
- board text added: "RAM"
- board text added: "ROM"
- board text removed: "EMM for X1"

Commit message: Add files via upload
Parts:
- D1, D2: value 1S4 -> 1N4148
Other:
- board text added: "1N4148"

Commit message: Add files via upload
Parts:
- removed C19: 0.1uF, Capacitor_THT:C_Rect_L4.0mm_W2.5mm_P2.50mm
- removed D3: 1S4, Diode_THT:D_DO-41_SOD81_P10.16mm_Horizontal
- removed U17: 74LS04, Package_DIP:DIP-14_W7.62mm_LongPads
- added Q1: 2N7000, Package_TO_SOT_THT:TO-92, F.Cu at (89.1, 159.7)
- R2: value 10k -> 1K
- R3: value 10k -> 10K
- moved R2 46.5 mm to (89.1, 169.8), turned to 180 degrees
- moved R3 37.8 mm to (99.3, 184.6), turned to 180 degrees
Connections:
- R2 pad 1: Net-(C14-Pad1) -> Net-(Q1-Pad3)
- R2 pad 2: Net-(R2-Pad2) -> Net-(BT1-Pad1)
- R3 pad 1: Net-(C14-Pad1) -> Net-(R3-Pad1)
- R3 pad 2: Net-(R3-Pad2) -> +5V
- S3 pad 1: Net-(D3-Pad1) -> /x3_WR
- S3 pad 2: Net-(R3-Pad2) -> Net-(R3-Pad1)
- U14 pad 22: Net-(R2-Pad2) -> Net-(Q1-Pad3)
- U14 pad 24: Net-(R2-Pad2) -> Net-(U12-Pad4)
- U14 pad 29: Net-(R3-Pad2) -> Net-(R3-Pad1)
Routing:
- net Net-(R2-Pad2): track 100.8 -> 0.00 mm, vias 3 -> 0
- net Net-(Q1-Pad3): track 0.00 -> 66.0 mm, vias 0 -> 1
- net Net-(R3-Pad2): track 60.4 -> 0.00 mm
- net Net-(R3-Pad1): track 0.00 -> 48.4 mm
- net /~RD: track 115.2 -> 160.8 mm, vias 1 -> 0
- net /x3_WR: track 79.6 -> 118.0 mm
- net Net-(D3-Pad1): track 35.2 -> 0.00 mm
- net Net-(U14-Pad5): track 94.4 -> 128.5 mm, vias 1 -> 0
- net Net-(U14-Pad6): track 99.1 -> 123.2 mm, vias 1 -> 0
- net Net-(D3-Pad2): track 22.8 -> 0.00 mm
- net Net-(C14-Pad1): track 49.0 -> 27.7 mm
- net +5V: track 554.9 -> 574.7 mm, vias 0 -> 1
- net Net-(U14-Pad8): track 110.8 -> 129.1 mm
- net /x3_RD: track 129.5 -> 146.5 mm
- net Net-(U14-Pad7): track 110.8 -> 127.5 mm
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Other:
- board text added: "10K"
- board text added: "1K"
- board text added: "2N7000"
- board text added: "EMM for X1 Rev1.8"
- board text removed: "1S4"
- board text removed: "EMM for X1 Rev1.5"
