File: Kicad/X1_EMM.sch (KiCad schematic (older format))
At the start: 42 parts, among them J1 for Card-Slot, U1 74LS04, U10 74LS193, U11 74LS193, U12 74LS138, U13 74LS138, U14 HM628512LFP-5, U15 74LS11, U16 74LS245, U2 74LS04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

Commit message: Add files via upload
Parts:
- added C19: 0.1uF, Capacitor_THT:C_Rect_L4.0mm_W2.5mm_P2.50mm, symbol Device:C
- added D3: 1S4, Diode_THT:D_DO-41_SOD81_P10.16mm_Horizontal, symbol Diode:1N4001
- added R3: 10k, Resistor_THT:R_Axial_DIN0207_L6.3mm_D2.5mm_P7.62mm_Horizontal, symbol Device:R
- added S3: SLIDE_SWITCH_3P, Connector_PinHeader_2.54mm:PinHeader_1x03_P2.54mm_Vertical, symbol Memory_RAM2:SLIDE_SWITCH_3P
- added U17: 74LS04, Package_DIP:DIP-14_W7.62mm_LongPads, symbol 74xx:74LS04
Connections:
- wire segments 497 -> 523
- no-connect marks 37 -> 40
Other:
- moved on the sheet: BT1, C1, C15, C2, C3, C4, C5, D1, D2, R2, U15D, U1G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

Commit message: Add files via upload
Parts:
- D1, D2: value 1S4 -> 1N4148
Changed lines of the file:
@@
 AR Path="/6938340F/69469E5D" Ref="D?"  Part="1"
 F 0 "D2" H 19850 8367 50  0000 C CNN
-F 1 "1S4" H 19850 8276 50  0000 C CNN
+F 1 "1N4148" H 19850 8276 50  0000 C CNN
 F 2 "Diode_THT:D_DO-41_SOD81_P10.16mm_Horizontal" H 19850 7975 50  0001 C CNN
 F 3 "http://www.vishay.com/docs/88503/1n4001.pdf" H 19850 8150 50  0001 C CNN
@@
 AR Path="/6938340F/69469E65" Ref="D?"  Part="1"
 F 0 "D1" H 18850 8417 50  0000 C CNN
-F 1 "1S4" H 18850 8326 50  0000 C CNN
+F 1 "1N4148" H 18850 8326 50  0000 C CNN
 F 2 "Diode_THT:D_DO-41_SOD81_P10.16mm_Horizontal" H 18850 8025 50  0001 C CNN
 F 3 "http://www.vishay.com/docs/88503/1n4001.pdf" H 18850 8200 50  0001 C CNN

Commit message: Add files via upload
Parts:
- removed C19: 0.1uF, Capacitor_THT:C_Rect_L4.0mm_W2.5mm_P2.50mm, symbol Device:C
- removed D3: 1S4, Diode_THT:D_DO-41_SOD81_P10.16mm_Horizontal, symbol Diode:1N4001
- removed U17: 74LS04, Package_DIP:DIP-14_W7.62mm_LongPads, symbol 74xx:74LS04
- added Q1: 2N7000, Package_TO_SOT_THT:TO-92, symbol Device:Q_NMOS_SGD
- R2: value 10k -> 1K
- R3: value 10k -> 10K
Connections:
- wire segments 523 -> 508
- no-connect marks 40 -> 36
Other:
- moved on the sheet: BT1, D1, D2
